File: HW/Version1/InterfazSensores.brd (EAGLE design)
At the start: 65.6 x 34.3 mm, 32 parts, among them IC1 LM2940, T1 BC846, T2 BC846, T3 BC846

Commit message: Placa finalizada
Revisada, lista para fabricar.
Parts:
- renumbered CENTRAL to J1, MAX485 to IC2, MICRO to IC3, SENSOR to J2, SV1 to BDM
Routing:
- net RST: track 15.7 -> 15.1 mm
- added copper zone on layer 16, net GND
- removed copper zone on layer 16, net N$11
