File: HW/Version1/InterfazSensores.brd (EAGLE design)
At the start: 65.6 x 34.3 mm, 32 parts, among them IC1 LM2940, IC2 LTC485S, IC3 SH8, J1 central, J2 sensor, T1 BC846, T2 BC846, T3 BC846

Commit message: Actualizo y agrego lista de materiales
Lista de materiales actualizada a travez del SCH
Parts:
- C4, C5: value 100n -> 100nF
- R1: value 4,7k-10k -> 10k
Changed lines of the file:
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@@
 <attribute name="VALUE" x="8.255" y="26.67" size="1.27" layer="27" rot="R270"/>
 </element>
-<element name="C4" library="resistor" package="C0805" value="100n" x="24.765" y="22.225" smashed="yes" rot="R180">
+<element name="C4" library="resistor" package="C0805" value="100nF" x="24.765" y="22.225" smashed="yes" rot="R180">
 <attribute name="NAME" x="24.13" y="23.495" size="1.27" layer="25"/>
 <attribute name="VALUE" x="26.035" y="24.765" size="1.27" layer="27" rot="R180"/>
 </element>
-<element name="C5" library="resistor" package="C0805" value="100n" x="20.955" y="16.51" smashed="yes" rot="R180">
+<element name="C5" library="resistor" package="C0805" value="100nF" x="20.955" y="16.51" smashed="yes" rot="R180">
 <attribute name="NAME" x="20.32" y="17.78" size="1.27" layer="25"/>
 <attribute name="VALUE" x="22.225" y="19.05" size="1.27" layer="27" rot="R180"/>
@@
 <attribute name="VALUE" x="32.004" y="25.654" size="1.27" layer="27" rot="R270"/>
 </element>
-<element name="R1" library="resistor" package="R0805" value="4,7k-10k" x="20.32" y="25.4" smashed="yes" rot="R180">
+<element name="R1" library="resistor" package="R0805" value="10k" x="20.32" y="25.4" smashed="yes" rot="R180">
 <attribute name="NAME" x="20.955" y="24.13" size="1.27" layer="25" rot="R180"/>
 <attribute name="VALUE" x="20.955" y="27.94" size="1.27" layer="27" rot="R180"/>
